File: unpad/usb.kicad_sch (KiCad schematic)
At the start: 1 part, among them J1 USB_C_Receptacle_USB2.0

Commit message: CREATE: primer intento de diseñar la pcb
Parts:
- removed J1: USB_C_Receptacle_USB2.0, symbol Connector:USB_C_Receptacle_USB2.0
Changed lines of the file:
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@@
 (kicad_sch (version 20230121) (generator eeschema)
   (paper "A4")
-  (symbol (lib_id "Connector:USB_C_Receptacle_USB2.0") (at 157.48 50.8 0) (unit 1)
-    (in_bom yes) (on_board yes) (dnp no) (fields_autoplaced)
-    (property "Reference" "J1" (at 157.48 27.94 0)
-      (effects (font (size 1.27 1.27)))
-    )
-    (property "Value" "USB_C_Receptacle_USB2.0" (at 157.48 30.48 0)
-      (effects (font (size 1.27 1.27)))
-    )
-    (property "Footprint" "" (at 161.29 50.8 0)
-      (effects (font (size 1.27 1.27)) hide)
-    )
-    (property "Datasheet" "https://www.usb.org/sites/default/files/documents/usb_type-c.zip" (at 161.29 50.8 0)
-      (effects (font (size 1.27 1.27)) hide)
-    )
-    (pin "A1")
-    (pin "A12")
-    (pin "A4")
-    (pin "A5")
-    (pin "A6")
-    (pin "A7")
-    (pin "A8")
-    (pin "A9")
-    (pin "B1")
-    (pin "B12")
-    (pin "B4")
-    (pin "B5")
-    (pin "B6")
-    (pin "B7")
-    (pin "B8")
-    (pin "B9")
-    (pin "S1")
-    (instances
-      (project "unpad"
-        (path "/ab6dd771-6418-466f-9873-5519077610f0/6f443b43-a46e-4c6a-a7f1-eeb518dc53e2"
-          (reference "J1") (unit 1)
-        )
-      )
-    )
-  )
   (symbol (lib_id "power:GND") (at 157.48 73.66 0) (unit 1)
     (in_bom yes) (on_board yes) (dnp no) (fields_autoplaced)
